File: src/osr_elec/elec/layout/rpi-hat/rpi-hat.kicad_pcb (KiCad board)
At the start: 4 copper layers, 85 x 56.5 mm, 4 parts

Commit message: wip: layout
Parts:
- added C1: 25V 10uF X5R ±10% 0805 Multilayer Ceramic Capacitors MLCC -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, lib:C0805, F.Cu at (161.1, 82.7)
- added C10: ?, lib:C0603, F.Cu at (210.1, 74.4)
- added C11: 50V 100nF X7R ±10% 0603 Multilayer Ceramic Capacitors MLCC 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, lib:C0603, F.Cu at (214.3, 52.4)
- added C12: 50V 100nF X7R ±10% 0603 Multilayer Ceramic Capacitors MLCC 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, lib:C0603, F.Cu at (75.1, 76.2)
- added C13: 50V 100nF X7R ±10% 0603 Multilayer Ceramic Capacitors MLCC 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, lib:C0603, F.Cu at (95.1, 59.4)
- added C14: 16V 4.7uF X5R ±10% 0603 Multilayer Ceramic Capacitors MLCC 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, lib:C0603, F.Cu at (91.3, 78.1)
- added C15: 50V 100nF X7R ±10% 0603 Multilayer Ceramic Capacitors MLCC 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, lib:C0603, F.Cu at (95.1, 63.9)
- added C16: 16V 4.7uF X5R ±10% 0603 Multilayer Ceramic Capacitors MLCC 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, lib:C0603, F.Cu at (91.3, 73.1)
- added C17: 50V 10nF X7R ±10% 0402 Multilayer Ceramic Capacitors MLCC -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, lib:C0402, F.Cu at (94.6, 68.2)
- added C18: 25V 1uF X5R ±10% 0402 Multilayer Ceramic Capacitors MLCC - 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, lib:C0402, F.Cu at (74.5, 80.5)
- added C2: 25V 10uF X5R ±10% 0805 Multilayer Ceramic Capacitors MLCC -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, lib:C0805, F.Cu at (151.1, 80.0)
- added C3: 50V 100nF X7R ±10% 0603 Multilayer Ceramic Capacitors MLCC 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, lib:C0603, F.Cu at (194.2, 63.2)
- added C4: 50V 100nF X7R ±10% 0603 Multilayer Ceramic Capacitors MLCC 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, lib:C0603, F.Cu at (248.6, 75.7)
- added C5: ?, lib:C0603, F.Cu at (249.4, 84.5)
- added C6: ?, lib:C0603, F.Cu at (249.3, 78.6)
- added C7: 50V 100nF X7R ±10% 0603 Multilayer Ceramic Capacitors MLCC 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, lib:C0603, F.Cu at (233.4, 95.2)
- added C8: 50V 100nF X7R ±10% 0603 Multilayer Ceramic Capacitors MLCC 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, lib:C0603, F.Cu at (200.3, 56.1)
- added C9: ?, lib:C0603, F.Cu at (208.1, 71.0)
- added D1: ?, LED_SMD:LED_0603_1608Metric, F.Cu at (164.7, 75.9)
- added D2: ?, LED_SMD:LED_0603_1608Metric, F.Cu at (169.2, 87.1)
- added D3: ?, LED_SMD:LED_0603_1608Metric, F.Cu at (168.5, 34.7)
- added D4: ?, LED_SMD:LED_0603_1608Metric, F.Cu at (190.2, 81.1)
- added D5: ?, LED_SMD:LED_0603_1608Metric, F.Cu at (181.9, 74.3)
- added D6: ?, LED_SMD:LED_0603_1608Metric, F.Cu at (181.9, 71.1)
- added D7: ?, LED_SMD:LED_0603_1608Metric, F.Cu at (208.7, 48.5)
- added D8: ?, LED_SMD:LED_0603_1608Metric, F.Cu at (203.5, 68.8)
- added D9: ?, LED_SMD:LED_0603_1608Metric, F.Cu at (200.5, 68.8)
- added FD1: ?, Fiducial:Fiducial_0.75mm_Mask1.5mm, F.Cu at (123.1, 108.3)
- added FD2: ?, Fiducial:Fiducial_0.75mm_Mask1.5mm, F.Cu at (127.0, 108.2)
- added FD3: ?, Fiducial:Fiducial_0.75mm_Mask1.5mm, F.Cu at (130.5, 108.2)
- added FD4: ?, Fiducial:Fiducial_0.75mm_Mask1.5mm, F.Cu at (133.7, 108.4)
- added J1: ?, lib:Combo__AMASS_XT30PW-M_1x02_P2.50mm_Horizontal__TerminalBlock_Phoenix_PT-1,5-2-5.0-H_1x02_P5.00mm_Horizontal, F.Cu at (153.4, 87.2)
- added J10: ?, Connector_PinHeader_2.54mm:PinHeader_1x05_P2.54mm_Vertical, F.Cu at (148.9, 55.7)
- added J11: ?, Connector_PinHeader_2.54mm:PinHeader_1x05_P2.54mm_Vertical, F.Cu at (75.0, 70.9)
- added J2: ?, lib:PinSocket_Samtec_ESQ-120-23-T-D_Oval_Pads, B.Cu at (150.0, 50.0)
- added J3: ?, Connector_PinHeader_2.54mm:PinHeader_1x03_P2.54mm_Vertical, F.Cu at (144.8, 55.6)
- added J4: ?, Connector_PinHeader_2.54mm:PinHeader_1x02_P2.54mm_Vertical, F.Cu at (194.6, 66.5)
- added J5: ?, Connector_JST:JST_PH_B2B-PH-K_1x02_P2.00mm_Vertical, F.Cu at (163.0, 34.8)
- added J6: ?, Connector_PinHeader_2.54mm:PinHeader_1x03_P2.54mm_Vertical, F.Cu at (177.5, 74.7)
- added J7: ?, TerminalBlock_Phoenix:TerminalBlock_Phoenix_PT-1,5-3-3.5-H_1x03_P3.50mm_Horizontal, F.Cu at (231.6, 109.6)
- added J8: ?, Connector_JST:JST_GH_SM04B-GHS-TB_1x04-1MP_P1.25mm_Horizontal, F.Cu at (222.1, 56.3)
- added J9: ?, Connector_JST:JST_GH_SM04B-GHS-TB_1x04-1MP_P1.25mm_Horizontal, F.Cu at (222.2, 67.3)
- added Q1: ?, Package_TO_SOT_SMD:SOT-23-3, F.Cu at (157.7, 58.8)
- added Q2: ?, Package_TO_SOT_SMD:SOT-23-3, F.Cu at (176.8, 29.3)
- added R1: 100mW Thick Film Resistors 75V ±100ppm/℃ ±1% 10kΩ 0603 Chip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, lib:R0603, F.Cu at (152.5, 61.1)
- added R10: 100mW Thick Film Resistors 75V ±100ppm/℃ ±1% 402Ω 0603 Chip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, lib:R0603, F.Cu at (168.5, 31.5)
- added R11: 100mW Thin Film Resistor 75V ±25ppm/℃ ±0.1% 84.5Ω 0603 Chip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, lib:R0603, F.Cu at (190.2, 79.2)
- added R12: 100mW Thick Film Resistors 75V ±100ppm/℃ ±1% 330Ω 0603 Chip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, lib:R0603, F.Cu at (185.2, 74.4)
- added R13: 166.667mW Thin Film Resistor 75V ±0.5% ±25ppm/℃ 316Ω 0603 C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, lib:R0603, F.Cu at (185.2, 71.1)
- added R14: 100mW Thick Film Resistors 75V ±100ppm/℃ ±1% 20Ω 0603 Chip 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, lib:R0603, F.Cu at (245.7, 86.3)
- added R15: 100mW Thick Film Resistors 75V ±100ppm/℃ ±1% 20Ω 0603 Chip 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, lib:R0603, F.Cu at (234.4, 87.9)
- added R16: 100mW Thick Film Resistors 75V ±100ppm/℃ ±1% 10kΩ 0603 Chip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, lib:R0603, F.Cu at (237.4, 87.9)
- added R17: 100mW Thick Film Resistors 75V ±1% ±400ppm/℃ 10Ω 0603 Chip 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, lib:R0603, F.Cu at (230.4, 100.4)
- added R18: 100mW Thick Film Resistors 75V ±1% ±400ppm/℃ 10Ω 0603 Chip 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, lib:R0603, F.Cu at (235.8, 100.5)
- added R19: 100mW Thick Film Resistors 75V ±100ppm/℃ ±1% 120Ω 0603 Chip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, lib:R0603, F.Cu at (233.2, 104.8)
- added R2: 100mW Thick Film Resistors 75V ±100ppm/℃ ±1% 47kΩ 0603 Chip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, lib:R0603, F.Cu at (155.1, 61.4)
- added R20: 100mW Thin Film Resistor 75V ±25ppm/℃ ±0.1% 84.5Ω 0603 Chip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, lib:R0603, F.Cu at (209.1, 52.1)
- added R21: 100mW Thick Film Resistors 75V ±100ppm/℃ ±1% 330Ω 0603 Chip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, lib:R0603, F.Cu at (203.6, 64.6)
- added R22: 166.667mW Thin Film Resistor 75V ±0.5% ±25ppm/℃ 316Ω 0603 C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, lib:R0603, F.Cu at (200.5, 64.7)
- added R23: 100mW Thick Film Resistors 75V ±100ppm/℃ ±1% 120Ω 0603 Chip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, lib:R0603, F.Cu at (218.1, 64.4)
- added R3: 100mW Thick Film Resistors 75V ±100ppm/℃ ±1% 1kΩ 0603 Chip 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, lib:R0603, F.Cu at (189.1, 65.6)
- added R4: 100mW Thick Film Resistors 75V ±100ppm/℃ ±1% 3.3kΩ 0603 Chi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, lib:R0603, F.Cu at (192.1, 54.7)
- added R5: 100mW Thick Film Resistors 75V ±100ppm/℃ ±1% 3.3kΩ 0603 Chi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, lib:R0603, F.Cu at (188.5, 56.2)
- added R6: 100mW Thick Film Resistors 75V ±100ppm/℃ ±1% 226Ω 0603 Chip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, lib:R0603, F.Cu at (166.5, 76.0)
- added R7: 100mW Thick Film Resistors ±100ppm/℃ ±1% 487Ω 0603 Chip Res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, lib:R0603, F.Cu at (169.6, 84.0)
- added R8: 100mW Thick Film Resistors 75V ±1% ±200ppm/℃ 100Ω 0603 Chip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, lib:R0603, F.Cu at (172.2, 28.5)
- added R9: 100mW Thick Film Resistors 75V ±100ppm/℃ ±1% 1MΩ 0603 Chip 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, lib:R0603, F.Cu at (172.1, 32.0)
- added S1: ?, lib:CK_JS102011JCQN_SW_SPDT_Slide_SMD, F.Cu at (214.7, 67.3)
- added TP1: ?, lib:Koa_Speer_RCWCTE_test_point, F.Cu at (145.4, 91.4)
- added TP2: ?, lib:Koa_Speer_RCWCTE_test_point, F.Cu at (145.2, 85.5)
- added TP3: ?, lib:Koa_Speer_RCWCTE_test_point, F.Cu at (161.4, 76.1)
- added TP4: ?, lib:Koa_Speer_RCWCTE_test_point, F.Cu at (166.5, 87.2)
- added U1: ?, Package_TO_SOT_SMD:SOT-23-6, F.Cu at (153.6, 57.6)
- added U10: ?, Package_QFP:LQFP-32_7x7mm_P0.8mm, F.Cu at (66.1, 65.6)
- added U2: ?, lib:SOT-223-3_L6.5-W3.4-P2.30-LS7.0-BR, F.Cu at (156.0, 79.7)
- added U3: ?, Package_SO:SOIC-8_3.9x4.9mm_P1.27mm, F.Cu at (194.2, 58.5)
- added U4: ?, Package_SO:TSSOP-28_4.4x9.7mm_P0.65mm, F.Cu at (197.9, 80.3)
- added U5: ?, Package_SO:SOIC-8_3.9x4.9mm_P1.27mm, F.Cu at (237.9, 93.9)
- added U6: ?, Package_TO_SOT_SMD:SOT-23-3, F.Cu at (233.2, 100.3)
- added U7: ?, Package_SO:SOIC-14_3.9x8.7mm_P1.27mm, F.Cu at (206.1, 58.3)
- added U8: ?, Package_SO:SOIC-8_3.9x4.9mm_P1.27mm, F.Cu at (214.8, 57.9)
- added U9: ?, lib:HDR-SMD_10P-P1.27-V-M-R2-C5-LS5.3, F.Cu at (66.8, 55.4)
- added X1: ?, Crystal:Crystal_SMD_Abracon_ABM8G-4Pin_3.2x2.5mm, F.Cu at (249.5, 81.5)
- added X2: ?, Crystal:Crystal_SMD_Abracon_ABM8G-4Pin_3.2x2.5mm, F.Cu at (208.2, 66.8)
