File: src/osr_elec/elec/layout/rpi-hat/rpi-hat.kicad_pcb (KiCad board)
At the start: 4 copper layers, 85 x 56.5 mm, 4 parts

Commit message: wip: layout
Parts:
- added C1: 25V 10uF X5R ±10% 0805 Multilayer Ceramic Capacitors MLCC -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, lib:C0805, F.Cu at (161.1, 82.7)
- added C10: 13.2 to 22.8 pF, lib:C0603, F.Cu at (254.5, 50.0)
- added C11: 50V 100nF X7R ±10% 0603 Multilayer Ceramic Capacitors MLCC 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, lib:C0603, F.Cu at (252.2, 69.3)
- added C2: 25V 10uF X5R ±10% 0805 Multilayer Ceramic Capacitors MLCC -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, lib:C0805, F.Cu at (151.1, 80.0)
- added C3: 50V 100nF X7R ±10% 0603 Multilayer Ceramic Capacitors MLCC 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, lib:C0603, F.Cu at (96.8, 65.9)
- added C4: 50V 100nF X7R ±10% 0603 Multilayer Ceramic Capacitors MLCC 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, lib:C0603, F.Cu at (256.4, 94.4)
- added C5: 13.2 to 22.8 pF, lib:C0603, F.Cu at (236.7, 96.6)
- added C6: 13.2 to 22.8 pF, lib:C0603, F.Cu at (245.4, 100.8)
- added C7: 50V 100nF X7R ±10% 0603 Multilayer Ceramic Capacitors MLCC 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, lib:C0603, F.Cu at (173.9, 27.5)
- added C8: 50V 100nF X7R ±10% 0603 Multilayer Ceramic Capacitors MLCC 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, lib:C0603, F.Cu at (248.9, 37.5)
- added C9: 13.2 to 22.8 pF, lib:C0603, F.Cu at (255.2, 45.5)
- added D1: , LED_SMD:LED_0603_1608Metric, F.Cu at (164.7, 75.9)
- added D2: , LED_SMD:LED_0603_1608Metric, F.Cu at (169.2, 87.1)
- added D3: , LED_SMD:LED_0603_1608Metric, F.Cu at (180.9, 155.1)
- added D4: , LED_SMD:LED_0603_1608Metric, F.Cu at (241.0, 112.3)
- added D5: , LED_SMD:LED_0603_1608Metric, F.Cu at (245.4, 113.2)
- added D6: , LED_SMD:LED_0603_1608Metric, F.Cu at (250.9, 112.4)
- added D7: , LED_SMD:LED_0603_1608Metric, F.Cu at (256.4, 64.6)
- added D8: , LED_SMD:LED_0603_1608Metric, F.Cu at (245.1, 26.9)
- added D9: , LED_SMD:LED_0603_1608Metric, F.Cu at (243.8, 33.0)
- added FD1: , Fiducial:Fiducial_0.75mm_Mask1.5mm, F.Cu at (123.1, 108.3)
- added FD2: , Fiducial:Fiducial_0.75mm_Mask1.5mm, F.Cu at (127.0, 108.2)
- added FD3: , Fiducial:Fiducial_0.75mm_Mask1.5mm, F.Cu at (130.5, 108.2)
- added FD4: , Fiducial:Fiducial_0.75mm_Mask1.5mm, F.Cu at (133.7, 108.4)
- added J1: , lib:Combo__AMASS_XT30PW-M_1x02_P2.50mm_Horizontal__TerminalBlock_Phoenix_PT-1,5-2-5.0-H_1x02_P5.00mm_Horizontal, F.Cu at (153.4, 87.2)
- added J10: , Connector_PinHeader_2.54mm:PinHeader_1x05_P2.54mm_Vertical, F.Cu at (160.2, 54.4)
- added J2: , lib:PinSocket_Samtec_ESQ-120-23-T-D_Oval_Pads, B.Cu at (150.0, 50.0)
- added J3: , Connector_PinHeader_2.54mm:PinHeader_1x03_P2.54mm_Vertical, F.Cu at (144.8, 55.6)
- added J4: , Connector_PinHeader_2.54mm:PinHeader_1x02_P2.54mm_Vertical, F.Cu at (97.6, 72.2)
- added J5: , Connector_JST:JST_PH_B2B-PH-K_1x02_P2.00mm_Vertical, F.Cu at (174.4, 147.5)
- added J6: , Connector_PinHeader_2.54mm:PinHeader_1x03_P2.54mm_Vertical, F.Cu at (240.0, 101.4)
- added J7: , TerminalBlock_Phoenix:TerminalBlock_Phoenix_PT-1,5-3-3.5-H_1x03_P3.50mm_Horizontal, F.Cu at (155.8, 24.4)
- added J8: , Connector_JST:JST_GH_SM04B-GHS-TB_1x04-1MP_P1.25mm_Horizontal, F.Cu at (247.0, 43.1)
- added J9: , Connector_JST:JST_GH_SM04B-GHS-TB_1x04-1MP_P1.25mm_Horizontal, F.Cu at (246.7, 52.6)
- added Q1: , Package_TO_SOT_SMD:SOT-23-3, F.Cu at (156.8, 64.8)
- added Q2: , Package_TO_SOT_SMD:SOT-23-3, F.Cu at (189.8, 153.5)
- added R1: 100mW Thick Film Resistors 75V ±100ppm/℃ ±1% 10kΩ 0603 Chip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, lib:R0603, F.Cu at (162.9, 69.4)
- added R10: 100mW Thick Film Resistors 75V ±100ppm/℃ ±1% 402Ω 0603 Chip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, lib:R0603, F.Cu at (183.0, 149.1)
- added R11: 100mW Thin Film Resistor 75V ±25ppm/℃ ±0.1% 84.5Ω 0603 Chip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, lib:R0603, F.Cu at (252.8, 98.5)
- added R12: 100mW Thick Film Resistors 75V ±100ppm/℃ ±1% 330Ω 0603 Chip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, lib:R0603, F.Cu at (256.1, 105.2)
- added R13: 100mW Thick Film Resistors 75V ±100ppm/℃ ±1% 316Ω 0603 Chip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, lib:R0603, F.Cu at (254.7, 109.8)
- added R14: 100mW Thick Film Resistors 75V ±100ppm/℃ ±1% 20Ω 0603 Chip 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, lib:R0603, F.Cu at (160.6, 38.5)
- added R15: 100mW Thick Film Resistors 75V ±100ppm/℃ ±1% 20Ω 0603 Chip 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, lib:R0603, F.Cu at (161.4, 33.8)
- added R16: 100mW Thick Film Resistors 75V ±100ppm/℃ ±1% 10kΩ 0603 Chip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, lib:R0603, F.Cu at (173.8, 21.9)
- added R17: 100mW Thick Film Resistors 75V ±1% ±400ppm/℃ 10Ω 0603 Chip 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, lib:R0603, F.Cu at (155.3, 33.2)
- added R18: 100mW Thick Film Resistors 75V ±1% ±400ppm/℃ 10Ω 0603 Chip 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, lib:R0603, F.Cu at (185.6, 25.0)
- added R19: 100mW Thick Film Resistors 75V ±100ppm/℃ ±1% 120Ω 0603 Chip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, lib:R0603, F.Cu at (201.1, 29.6)
- added R2: 100mW Thick Film Resistors 75V ±100ppm/℃ ±1% 47kΩ 0603 Chip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, lib:R0603, F.Cu at (151.5, 69.3)
- added R20: 100mW Thin Film Resistor 75V ±25ppm/℃ ±0.1% 84.5Ω 0603 Chip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, lib:R0603, F.Cu at (256.7, 68.1)
- added R21: 100mW Thick Film Resistors 75V ±100ppm/℃ ±1% 330Ω 0603 Chip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, lib:R0603, F.Cu at (250.6, 29.1)
- added R22: 100mW Thick Film Resistors 75V ±100ppm/℃ ±1% 316Ω 0603 Chip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, lib:R0603, F.Cu at (247.8, 33.8)
- added R23: 100mW Thick Film Resistors 75V ±100ppm/℃ ±1% 120Ω 0603 Chip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, lib:R0603, F.Cu at (246.5, 69.1)
- added R3: 100mW Thick Film Resistors 75V ±100ppm/℃ ±1% 1kΩ 0603 Chip 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, lib:R0603, F.Cu at (96.4, 51.5)
- added R4: 100mW Thick Film Resistors 75V ±100ppm/℃ ±1% 3.3kΩ 0603 Chi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, lib:R0603, F.Cu at (103.1, 70.2)
- added R5: 100mW Thick Film Resistors 75V ±100ppm/℃ ±1% 3.3kΩ 0603 Chi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, lib:R0603, F.Cu at (102.2, 65.9)
- added R6: 100mW Thick Film Resistors 75V ±100ppm/℃ ±1% 226Ω 0603 Chip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, lib:R0603, F.Cu at (166.5, 76.0)
- added R7: 100mW Thick Film Resistors ±100ppm/℃ ±1% 487Ω 0603 Chip Res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, lib:R0603, F.Cu at (171.8, 87.1)
- added R8: 100mW Thick Film Resistors 75V ±1% ±200ppm/℃ 100Ω 0603 Chip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, lib:R0603, F.Cu at (185.3, 162.8)
- added R9: 100mW Thick Film Resistors 75V ±100ppm/℃ ±1% 1MΩ 0603 Chip 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, lib:R0603, F.Cu at (193.9, 163.5)
- added S1: , lib:CK_JS102011JCQN_SW_SPDT_Slide_SMD, F.Cu at (246.7, 61.9)
- added TP1: , lib:Koa_Speer_RCWCTE_test_point, F.Cu at (145.4, 91.4)
- added TP2: , lib:Koa_Speer_RCWCTE_test_point, F.Cu at (145.2, 85.5)
- added TP3: , lib:Koa_Speer_RCWCTE_test_point, F.Cu at (161.4, 76.1)
- added TP4: , lib:Koa_Speer_RCWCTE_test_point, F.Cu at (166.5, 87.2)
- added U1: , Package_TO_SOT_SMD:SOT-23-6, F.Cu at (162.9, 62.3)
- added U2: , lib:SOT-223-3_L6.5-W3.4-P2.30-LS7.0-BR, F.Cu at (156.0, 79.7)
- added U3: , Package_SO:SOIC-8_3.9x4.9mm_P1.27mm, F.Cu at (100.7, 57.1)
- added U4: , Package_SO:TSSOP-28_4.4x9.7mm_P0.65mm, F.Cu at (181.7, 57.9)
- added U5: , Package_SO:SOIC-8_3.9x4.9mm_P1.27mm, F.Cu at (193.2, 20.0)
- added U6: , Package_TO_SOT_SMD:SOT-23-3, F.Cu at (203.1, 19.2)
- added U7: , Package_SO:SOIC-14_3.9x8.7mm_P1.27mm, F.Cu at (257.9, 30.6)
- added U8: , Package_SO:SOIC-8_3.9x4.9mm_P1.27mm, F.Cu at (257.6, 57.7)
- added X1: , Crystal:Crystal_SMD_Abracon_ABM8G-4Pin_3.2x2.5mm, F.Cu at (249.3, 106.4)
- added X2: , Crystal:Crystal_SMD_Abracon_ABM8G-4Pin_3.2x2.5mm, F.Cu at (255.9, 40.5)
